File: kicad/midi_din_sync/midi_din_sync.kicad_pcb (KiCad board)
At the start: 2 copper layers, 70 x 60 mm, 6 parts, among them J1 DIN-5_180degree, J2 DIN-5_180degree, J3 DIN-5_180degree, J4 DIN-5_180degree, U1 6N138, U2 ProMicro

Commit message: Working on schematic and PCB
Parts:
- added C1: 0.1u, Capacitor_SMD:C_0805_2012Metric_Pad1.18x1.45mm_HandSolder, B.Cu at (141.0, 102.0)
- added D1: BAS316, Diode_SMD:D_SOD-323, B.Cu at (149.0, 115.0)
- added D2: LED, Connector_PinSocket_2.54mm:PinSocket_1x02_P2.54mm_Vertical, F.Cu at (129.0, 112.0)
- added D3: LED, Connector_PinSocket_2.54mm:PinSocket_1x02_P2.54mm_Vertical, F.Cu at (159.0, 112.0)
- added D4: LED, Connector_PinSocket_2.54mm:PinSocket_1x02_P2.54mm_Vertical, F.Cu at (129.0, 88.0)
- added D5: LED, Connector_PinSocket_2.54mm:PinSocket_1x02_P2.54mm_Vertical, F.Cu at (159.0, 88.0)
- added D6: LED, Connector_PinSocket_2.54mm:PinSocket_1x02_P2.54mm_Vertical, F.Cu at (115.0, 86.0)
- added R1: 220, Resistor_SMD:R_0805_2012Metric_Pad1.20x1.40mm_HandSolder, B.Cu at (168.0, 112.0)
- added R10: 470, Resistor_SMD:R_0805_2012Metric_Pad1.20x1.40mm_HandSolder, B.Cu at (116.0, 80.0)
- added R2: 220, Resistor_SMD:R_0805_2012Metric_Pad1.20x1.40mm_HandSolder, B.Cu at (139.0, 114.0)
- added R3: 220, Resistor_SMD:R_0805_2012Metric_Pad1.20x1.40mm_HandSolder, B.Cu at (152.0, 122.0)
- added R4: 470, Resistor_SMD:R_0805_2012Metric_Pad1.20x1.40mm_HandSolder, B.Cu at (146.0, 98.0)
- added R5: 10k, Resistor_SMD:R_0805_2012Metric_Pad1.20x1.40mm_HandSolder, B.Cu at (152.0, 98.0)
- added R6: 470, Resistor_SMD:R_0805_2012Metric_Pad1.20x1.40mm_HandSolder, B.Cu at (122.0, 112.0)
- added R7: 470, Resistor_SMD:R_0805_2012Metric_Pad1.20x1.40mm_HandSolder, B.Cu at (159.0, 107.0)
- added R8: 470, Resistor_SMD:R_0805_2012Metric_Pad1.20x1.40mm_HandSolder, B.Cu at (127.0, 80.0)
- added R9: 470, Resistor_SMD:R_0805_2012Metric_Pad1.20x1.40mm_HandSolder, B.Cu at (153.0, 89.0)
- moved U1 18.3 mm to (145.2, 110.8), turned to 90 degrees
Connections:
- J1 pad 4: unconnected-(J1-Pad4) -> Net-(J1-Pad4)
- J1 pad 5: unconnected-(J1-Pad5) -> Net-(U1-Pad3)
- J2 pad 2: unconnected-(J2-Pad2) -> GND
- J2 pad 4: unconnected-(J2-Pad4) -> Net-(J2-Pad4)
- J2 pad 5: unconnected-(J2-Pad5) -> Net-(J2-Pad5)
- J3 pad 2: unconnected-(J3-Pad2) -> GND
- J4 pad 2: unconnected-(J4-Pad2) -> GND
- U1 pad 2: unconnected-(U1-Pad2) -> Net-(U1-Pad2)
- U1 pad 3: unconnected-(U1-Pad3) -> Net-(U1-Pad3)
- U1 pad 5: unconnected-(U1-Pad5) -> GND
- U1 pad 6: unconnected-(U1-Pad6) -> RX
- U1 pad 7: unconnected-(U1-Pad7) -> Net-(U1-Pad7)
- U1 pad 8: unconnected-(U1-Pad8) -> +5V
- U2 pad 1: unconnected-(U2-Pad1) -> TX
- U2 pad 2: unconnected-(U2-Pad2) -> RX
Routing:
- net TX: track 0.00 -> 47.5 mm
- net RX: track 0.00 -> 45.6 mm
- net Net-(U1-Pad3): track 0.00 -> 33.9 mm
- net Net-(U1-Pad7): track 0.00 -> 20.6 mm
- net Net-(U1-Pad2): track 0.00 -> 12.5 mm
- net +5V: track 0.00 -> 9.52 mm
- net Net-(D4-Pad1): track 0.00 -> 7.83 mm
- net Net-(J2-Pad5): track 0.00 -> 7.78 mm
- net Net-(D6-Pad1): track 0.00 -> 6.00 mm
- net Net-(D5-Pad1): track 0.00 -> 5.41 mm
- net GND: track 0.00 -> 5.25 mm
- net Net-(D3-Pad1): track 0.00 -> 4.00 mm
- net Net-(J2-Pad4): track 0.00 -> 3.85 mm
- net Net-(J1-Pad4): track 0.00 -> 3.43 mm
- added copper zone on B.Cu, net GND

Commit message: Minor movements
Parts:
- added R11: 10k, Resistor_SMD:R_0805_2012Metric_Pad1.20x1.40mm_HandSolder, B.Cu at (147.0, 87.0)
- added R12: 220, Resistor_SMD:R_0805_2012Metric_Pad1.20x1.40mm_HandSolder, B.Cu at (133.0, 80.0)
- added R13: 220, Resistor_SMD:R_0805_2012Metric_Pad1.20x1.40mm_HandSolder, B.Cu at (148.0, 83.0)
- added R14: 220, Resistor_SMD:R_0805_2012Metric_Pad1.20x1.40mm_HandSolder, B.Cu at (138.0, 87.0)
- added R15: 220, Resistor_SMD:R_0805_2012Metric_Pad1.20x1.40mm_HandSolder, B.Cu at (172.0, 83.0)
- added R16: 10k, Resistor_SMD:R_0805_2012Metric_Pad1.20x1.40mm_HandSolder, B.Cu at (173.0, 87.0)
- moved R8 10.0 mm to (121.0, 88.0), turned to 0 degrees
- moved R7 9.06 mm to (158.0, 116.0), turned to 90 degrees
- moved R5 2.83 mm to (154.0, 100.0), turned to 0 degrees
- moved R4 2.00 mm to (146.0, 100.0)
- moved U2 1.80 mm to (127.8, 100.0)
- moved R2 1.63 mm to (140.6, 114.3)
Connections:
- D2 pad 2: unconnected-(D2-Pad2) -> MIDI_IN_LED
- D3 pad 2: unconnected-(D3-Pad2) -> MIDI_OUT_LED
- D4 pad 2: unconnected-(D4-Pad2) -> SYNC_OUT_LED
- D5 pad 2: unconnected-(D5-Pad2) -> SYNC_IN_LED
- D6 pad 2: unconnected-(D6-Pad2) -> POWER_LED
- J3 pad 1: unconnected-(J3-Pad1) -> Net-(J3-Pad1)
- J3 pad 3: unconnected-(J3-Pad3) -> Net-(J3-Pad3)
- J4 pad 1: unconnected-(J4-Pad1) -> Net-(J4-Pad1)
- J4 pad 3: unconnected-(J4-Pad3) -> Net-(J4-Pad3)
- U2 pad 13: unconnected-(U2-Pad13) -> CLOCK_IN
- U2 pad 14: unconnected-(U2-Pad14) -> START_IN
- U2 pad 15: unconnected-(U2-Pad15) -> CLOCK_OUT
- U2 pad 16: unconnected-(U2-Pad16) -> START_OUT
- U2 pad 17: unconnected-(U2-Pad17) -> SYNC_OUT_LED
- U2 pad 18: unconnected-(U2-Pad18) -> SYNC_IN_LED
- U2 pad 19: unconnected-(U2-Pad19) -> MIDI_OUT_LED
- U2 pad 20: unconnected-(U2-Pad20) -> MIDI_IN_LED
- U2 pad 21: unconnected-(U2-Pad21) -> POWER_LED
- U2 pad 24: unconnected-(U2-Pad24) -> +5V
- U2 pad 3: unconnected-(U2-Pad3) -> GND
- U2 pad 4: unconnected-(U2-Pad4) -> GND
Routing:
- net +5V: track 9.52 -> 84.4 mm, vias 0 -> 4
- net MIDI_OUT_LED: track 0.00 -> 50.1 mm
- net MIDI_IN_LED: track 0.00 -> 42.2 mm, vias 0 -> 2
- net SYNC_IN_LED: track 0.00 -> 38.0 mm, vias 0 -> 2
- net CLOCK_IN: track 0.00 -> 35.5 mm
- net Net-(J3-Pad1): track 0.00 -> 16.0 mm
- net START_IN: track 0.00 -> 15.1 mm
- net START_OUT: track 0.00 -> 11.9 mm
- net Net-(R5-Pad2): track 20.6 -> 12.3 mm
- net POWER_LED: track 0.00 -> 8.04 mm
- net Net-(D2-Pad1): track 0.00 -> 6.00 mm
- net RX: track 45.6 -> 40.1 mm
- net CLOCK_OUT: track 0.00 -> 4.92 mm
- net Net-(J4-Pad3): track 0.00 -> 4.69 mm
- net Net-(J4-Pad1): track 0.00 -> 4.69 mm
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