File: kicad/midi_din_sync/midi_din_sync.kicad_sch (KiCad schematic)
At the start: 6 parts, among them J1 DIN-5_180degree, J2 DIN-5_180degree, J3 DIN-5_180degree, J4 DIN-5_180degree, U1 6N138, U2 ProMicro

Commit message: Working on schematic and PCB
Parts:
- added C1: 0.1u, Capacitor_SMD:C_0805_2012Metric_Pad1.18x1.45mm_HandSolder, symbol Device:C_Small
- added D1: BAS316, Diode_SMD:D_SOD-323, symbol Diode:BAS316
- added D2, D3, D4, D5, D6: LED, Connector_PinSocket_2.54mm:PinSocket_1x02_P2.54mm_Vertical, symbol Device:LED
- added R1, R2, R3, R? (x4): 220, Resistor_SMD:R_0805_2012Metric_Pad1.20x1.40mm_HandSolder, symbol Device:R
- added R10, R4, R6, R7, R8, R9: 470, Resistor_SMD:R_0805_2012Metric_Pad1.20x1.40mm_HandSolder, symbol Device:R
- added R5: 10k, Resistor_SMD:R_0805_2012Metric_Pad1.20x1.40mm_HandSolder, symbol Device:R
Connections:
- net at J1.4: now also R2.1
- net at J1.5: now also U1.3 (C2), D1.2 (A)
- net TX: now reaches U2.1 (TX)
- net TX: now also R3.2
- net CLOCK_IN: now reaches U2.13 (B6,10)
- net CLOCK_IN: now also R?.2
- net START_IN: now reaches U2.14 (B2,16)
- net START_IN: now also R?.1
- net CLOCK_OUT: now reaches U2.15 (B3,14)
- net CLOCK_OUT: now also R?.2
- net START_OUT: now reaches U2.16 (B1,15)
- net START_OUT: now also R?.1
- net RX: now reaches U2.2 (RX)
- net RX: now also U1.6 (VO2), R4.1
- net +5V: now reaches U2.24 (RAW)
- net +5V: now also U1.8 (VCC), C1.1, R1.1, R4.2
- net GND: now reaches U2.3 (GND)
- net GND: now also J2.2, J3.2, J4.2, U1.5 (GND), U2.4 (GND), C1.2, R10.1, R5.1, R6.1, R7.1, R8.1, R9.1
- net at J2.4: now also R1.2
- net at J2.5: now also R3.1
- net at J3.1: now also R?.2
- net at J3.3: now also R?.1
- net at J4.1: now also R?.2
- net at J4.3: now also R?.1
- net at U1.2 (C1): now also D1.1 (K), R2.2
- net at U1.7 (VO1): now also R5.2
- new net: D4.1 (K), R8.2
- new net: D6.1 (K), R10.2
- new net: D2.1 (K), R6.2
- new net: D5.1 (K), R9.2
- new net: D3.1 (K), R7.2
Other:
- moved on the sheet: J1, J2, J3, J4, U1, U2

Commit message: Minor movements
Parts:
- added R11, R16: (no value), Resistor_SMD:R_0805_2012Metric_Pad1.20x1.40mm_HandSolder, symbol Device:R
- gave numbers to parts that had none: 4
Connections:
- net CLOCK_IN: now also R16.2
- net GND: now also R11.1, R16.1
- net START_IN: now also R11.2
- net SYNC_OUT_LED: now reaches U2.17 (F7,A0)
- net SYNC_OUT_LED: now also D4.2 (A)
- net SYNC_IN_LED: now reaches U2.18 (F6,A1)
- net SYNC_IN_LED: now also D5.2 (A)
- net MIDI_OUT_LED: now reaches U2.19 (F5,A2)
- net MIDI_OUT_LED: now also D3.2 (A)
- net MIDI_IN_LED: now reaches U2.20 (F4,A3)
- net MIDI_IN_LED: now also D2.2 (A)
- net POWER_LED: now reaches U2.21 (VCC)
- net POWER_LED: now also D6.2 (A)
Other:
- moved on the sheet: D2, D3, D4, D5, D6, R10, R6, R7, R8, R9
